Commit message: fixed camera

File: src/arm_description/description/camera.xacro (robot description, xacro)
@@ -6,9 +6,9 @@
       xyz:='0 0 0'
       rpy:='0 0 0'
-      width:=640
-      height:=480
-      hfov:=1.047
+      width:=1280
+      height:=720
+      hfov:=1.547
       update_rate:=30
-      near_clip:=0.02
+      near_clip:=0.01
       far_clip:=10.0">
     <link name="${prefix}_link">
@@ -19,9 +19,14 @@
       </inertial>
       <visual>
+        <origin xyz="0 0 0" rpy="0 0 0"/>
         <geometry>
           <box size="0.03 0.03 0.02"/>
         </geometry>
+        <material name="Blue">
+          <color rgba="0 0 1 1"/>
+        </material>
       </visual>
       <collision>
+        <origin xyz="0 0 0" rpy="0 0 0"/>
         <geometry>
           <box size="0.03 0.03 0.02"/>

File: src/arm_description/description/so101.urdf.xacro (robot description, xacro)
@@ -328,11 +328,11 @@
   </gazebo>
   <xacro:camera_sensor
-    parent="gripper_frame_link"
+    parent="wrist_link"
     prefix="camera"
-    xyz="-0.020 0.00 -0.08"
-    rpy="0 0 0"
-    width="640"
-    height="480"
-    hfov="1.047"
+    xyz="-0.08 -0.05 0.02"
+    rpy="1.57 0.00 -1.02"
+    width="1280"
+    height="720"
+    hfov="1.5708"
     update_rate="30"/>
 </robot>
