Commit message: gazebo working

File: src/arm_description/description/so101.urdf.xacro (robot description, xacro)
@@ -21,5 +21,5 @@
       <origin xyz="-0.00636471 -9.94414e-05 -0.0024" rpy="1.5708 -1.67685e-15 1.5708"/>
       <geometry>
-        <mesh filename="package://arm_description/assets/base_motor_holder_so101_v1.stl"/>
+        <mesh filename="model://arm_description/assets/base_motor_holder_so101_v1.stl"/>
       </geometry>
       <material name="3d_printed"/>
@@ -28,5 +28,5 @@
       <origin xyz="-0.00636471 -9.94414e-05 -0.0024" rpy="1.5708 -1.67685e-15 1.5708"/>
       <geometry>
-        <mesh filename="package://arm_description/assets/base_motor_holder_so101_v1.stl"/>
+        <mesh filename="model://arm_description/assets/base_motor_holder_so101_v1.stl"/>
       </geometry>
     </collision>
@@ -35,5 +35,5 @@
       <origin xyz="-0.00636471 -8.97657e-09 -0.0024" rpy="1.5708 -2.78073e-29 1.5708"/>
       <geometry>
-        <mesh filename="package://arm_description/assets/base_so101_v2.stl"/>
+        <mesh filename="model://arm_description/assets/base_so101_v2.stl"/>
       </geometry>
       <material name="3d_printed"/>
@@ -42,5 +42,5 @@
       <origin xyz="-0.00636471 -8.97657e-09 -0.0024" rpy="1.5708 -2.78073e-29 1.5708"/>
       <geometry>
-        <mesh filename="package://arm_description/assets/base_so101_v2.stl"/>
+        <mesh filename="model://arm_description/assets/base_so101_v2.stl"/>
       </geometry>
     </collision>
@@ -49,5 +49,5 @@
       <origin xyz="0.0263353 -8.97657e-09 0.0437" rpy="-8.21148e-16 7.84513e-18 1.249e-15"/>
       <geometry>
-        <mesh filename="package://arm_description/assets/sts3215_03a_v1.stl"/>
+        <mesh filename="model://arm_description/assets/sts3215_03a_v1.stl"/>
       </geometry>
       <material name="sts3215"/>
@@ -56,5 +56,5 @@
       <origin xyz="0.0263353 -8.97657e-09 0.0437" rpy="-8.21148e-16 7.84513e-18 1.249e-15"/>
       <geometry>
-        <mesh filename="package://arm_description/assets/sts3215_03a_v1.stl"/>
+        <mesh filename="model://arm_description/assets/sts3215_03a_v1.stl"/>
       </geometry>
     </collision>
@@ -63,5 +63,5 @@
       <origin xyz="-0.0309827 -0.000199441 0.0474" rpy="1.5708 -1.35493e-14 1.5708"/>
       <geometry>
-        <mesh filename="package://arm_description/assets/waveshare_mounting_plate_so101_v2.stl"/>
+        <mesh filename="model://arm_description/assets/waveshare_mounting_plate_so101_v2.stl"/>
       </geometry>
       <material name="3d_printed"/>
@@ -70,5 +70,5 @@
       <origin xyz="-0.0309827 -0.000199441 0.0474" rpy="1.5708 -1.35493e-14 1.5708"/>
       <geometry>
-        <mesh filename="package://arm_description/assets/waveshare_mounting_plate_so101_v2.stl"/>
+        <mesh filename="model://arm_description/assets/waveshare_mounting_plate_so101_v2.stl"/>
       </geometry>
     </collision>
@@ -85,5 +85,5 @@
       <origin xyz="-0.0303992 0.000422241 -0.0417" rpy="1.5708 1.5708 0"/>
       <geometry>
-        <mesh filename="package://arm_description/assets/sts3215_03a_v1.stl"/>
+        <mesh filename="model://arm_description/assets/sts3215_03a_v1.stl"/>
       </geometry>
       <material name="sts3215"/>
@@ -92,5 +92,5 @@
       <origin xyz="-0.0303992 0.000422241 -0.0417" rpy="1.5708 1.5708 0"/>
       <geometry>
-        <mesh filename="package://arm_description/assets/sts3215_03a_v1.stl"/>
+        <mesh filename="model://arm_description/assets/sts3215_03a_v1.stl"/>
       </geometry>
     </collision>
@@ -99,5 +99,5 @@
       <origin xyz="-0.0675992 -0.000177759 0.0158499" rpy="1.5708 -1.5708 0"/>
       <geometry>
-        <mesh filename="package://arm_description/assets/motor_holder_so101_base_v1.stl"/>
+        <mesh filename="model://arm_description/assets/motor_holder_so101_base_v1.stl"/>
       </geometry>
       <material name="3d_printed"/>
@@ -106,5 +106,5 @@
       <origin xyz="-0.0675992 -0.000177759 0.0158499" rpy="1.5708 -1.5708 0"/>
       <geometry>
-        <mesh filename="package://arm_description/assets/motor_holder_so101_base_v1.stl"/>
+        <mesh filename="model://arm_description/assets/motor_holder_so101_base_v1.stl"/>
       </geometry>
     </collision>
@@ -113,5 +113,5 @@
       <origin xyz="0.0122008 2.22413e-05 0.0464" rpy="-1.5708 2.35221e-33 0"/>
       <geometry>
-        <mesh filename="package://arm_description/assets/rotation_pitch_so101_v1.stl"/>
+        <mesh filename="model://arm_description/assets/rotation_pitch_so101_v1.stl"/>
       </geometry>
       <material name="3d_printed"/>
@@ -120,5 +120,5 @@
       <origin xyz="0.0122008 2.22413e-05 0.0464" rpy="-1.5708 2.35221e-33 0"/>
       <geometry>
-        <mesh filename="package://arm_description/assets/rotation_pitch_so101_v1.stl"/>
+        <mesh filename="model://arm_description/assets/rotation_pitch_so101_v1.stl"/>
       </geometry>
     </collision>
@@ -135,5 +135,5 @@
       <origin xyz="-0.11257 -0.0155 0.0187" rpy="-3.14159 -5.27356e-16 -1.5708"/>
       <geometry>
-        <mesh filename="package://arm_description/assets/sts3215_03a_v1.stl"/>
+        <mesh filename="model://arm_description/assets/sts3215_03a_v1.stl"/>
       </geometry>
       <material name="sts3215"/>
@@ -142,5 +142,5 @@
       <origin xyz="-0.11257 -0.0155 0.0187" rpy="-3.14159 -5.27356e-16 -1.5708"/>
       <geometry>
-        <mesh filename="package://arm_description/assets/sts3215_03a_v1.stl"/>
+        <mesh filename="model://arm_description/assets/sts3215_03a_v1.stl"/>
       </geometry>
     </collision>
@@ -149,5 +149,5 @@
       <origin xyz="-0.065085 0.012 0.0182" rpy="3.14159 -0 -1.30911e-30"/>
       <geometry>
-        <mesh filename="package://arm_description/assets/upper_arm_so101_v1.stl"/>
+        <mesh filename="model://arm_description/assets/upper_arm_so101_v1.stl"/>
       </geometry>
       <material name="3d_printed"/>
@@ -156,5 +156,5 @@
       <origin xyz="-0.065085 0.012 0.0182" rpy="3.14159 -0 -1.30911e-30"/>
       <geometry>
-        <mesh filename="package://arm_description/assets/upper_arm_so101_v1.stl"/>
+        <mesh filename="model://arm_description/assets/upper_arm_so101_v1.stl"/>
       </geometry>
     </collision>
@@ -171,5 +171,5 @@
       <origin xyz="-0.0648499 -0.032 0.0182" rpy="3.14159 -0 6.67202e-31"/>
       <geometry>
-        <mesh filename="package://arm_description/assets/under_arm_so101_v1.stl"/>
+        <mesh filename="model://arm_description/assets/under_arm_so101_v1.stl"/>
       </geometry>
       <material name="3d_printed"/>
@@ -178,5 +178,5 @@
       <origin xyz="-0.0648499 -0.032 0.0182" rpy="3.14159 -0 6.67202e-31"/>
       <geometry>
-        <mesh filename="package://arm_description/assets/under_arm_so101_v1.stl"/>
+        <mesh filename="model://arm_description/assets/under_arm_so101_v1.stl"/>
       </geometry>
     </collision>
@@ -185,5 +185,5 @@
       <origin xyz="-0.0648499 -0.032 0.018" rpy="-3.14159 -2.55351e-15 -1.83387e-30"/>
       <geometry>
-        <mesh filename="package://arm_description/assets/motor_holder_so101_wrist_v1.stl"/>
+        <mesh filename="model://arm_description/assets/motor_holder_so101_wrist_v1.stl"/>
       </geometry>
       <material name="3d_printed"/>
@@ -192,5 +192,5 @@
       <origin xyz="-0.0648499 -0.032 0.018" rpy="-3.14159 -2.55351e-15 -1.83387e-30"/>
       <geometry>
-        <mesh filename="package://arm_description/assets/motor_holder_so101_wrist_v1.stl"/>
+        <mesh filename="model://arm_description/assets/motor_holder_so101_wrist_v1.stl"/>
       </geometry>
     </collision>
@@ -199,5 +199,5 @@
       <origin xyz="-0.1224 0.0052 0.0187" rpy="-3.14159 -7.88861e-31 -3.14159"/>
       <geometry>
-        <mesh filename="package://arm_description/assets/sts3215_03a_v1.stl"/>
+        <mesh filename="model://arm_description/assets/sts3215_03a_v1.stl"/>
       </geometry>
       <material name="sts3215"/>
@@ -206,5 +206,5 @@
       <origin xyz="-0.1224 0.0052 0.0187" rpy="-3.14159 -7.88861e-31 -3.14159"/>
       <geometry>
-        <mesh filename="package://arm_description/assets/sts3215_03a_v1.stl"/>
+        <mesh filename="model://arm_description/assets/sts3215_03a_v1.stl"/>
       </geometry>
     </collision>
@@ -221,5 +221,5 @@
       <origin xyz="8.32667e-17 -0.0424 0.0306" rpy="1.5708 1.5708 0"/>
       <geometry>
-        <mesh filename="package://arm_description/assets/sts3215_03a_no_horn_v1.stl"/>
+        <mesh filename="model://arm_description/assets/sts3215_03a_no_horn_v1.stl"/>
       </geometry>
       <material name="sts3215"/>
@@ -228,5 +228,5 @@
       <origin xyz="8.32667e-17 -0.0424 0.0306" rpy="1.5708 1.5708 0"/>
       <geometry>
-        <mesh filename="package://arm_description/assets/sts3215_03a_no_horn_v1.stl"/>
+        <mesh filename="model://arm_description/assets/sts3215_03a_no_horn_v1.stl"/>
       </geometry>
     </collision>
@@ -235,5 +235,5 @@
       <origin xyz="0 -0.028 0.0181" rpy="-1.5708 -1.5708 0"/>
       <geometry>
-        <mesh filename="package://arm_description/assets/wrist_roll_pitch_so101_v2.stl"/>
+        <mesh filename="model://arm_description/assets/wrist_roll_pitch_so101_v2.stl"/>
       </geometry>
       <material name="3d_printed"/>
@@ -242,5 +242,5 @@
       <origin xyz="0 -0.028 0.0181" rpy="-1.5708 -1.5708 0"/>
       <geometry>
-        <mesh filename="package://arm_description/assets/wrist_roll_pitch_so101_v2.stl"/>
+        <mesh filename="model://arm_description/assets/wrist_roll_pitch_so101_v2.stl"/>
       </geometry>
     </collision>
@@ -257,5 +257,5 @@
       <origin xyz="0.0077 0.0001 -0.0234" rpy="-1.5708 -5.19179e-17 -1.66533e-16"/>
       <geometry>
-        <mesh filename="package://arm_description/assets/sts3215_03a_v1.stl"/>
+        <mesh filename="model://arm_description/assets/sts3215_03a_v1.stl"/>
       </geometry>
       <material name="sts3215"/>
@@ -264,5 +264,5 @@
       <origin xyz="0.0077 0.0001 -0.0234" rpy="-1.5708 -5.19179e-17 -1.66533e-16"/>
       <geometry>
-        <mesh filename="package://arm_description/assets/sts3215_03a_v1.stl"/>
+        <mesh filename="model://arm_description/assets/sts3215_03a_v1.stl"/>
       </geometry>
     </collision>
@@ -271,5 +271,5 @@
       <origin xyz="8.32667e-17 -0.000218214 0.000949706" rpy="-3.14159 -5.55112e-17 0"/>
       <geometry>
-        <mesh filename="package://arm_description/assets/wrist_roll_follower_so101_v1.stl"/>
+        <mesh filename="model://arm_description/assets/wrist_roll_follower_so101_v1.stl"/>
       </geometry>
       <material name="3d_printed"/>
@@ -278,5 +278,5 @@
       <origin xyz="8.32667e-17 -0.000218214 0.000949706" rpy="-3.14159 -5.55112e-17 0"/>
       <geometry>
-        <mesh filename="package://arm_description/assets/wrist_roll_follower_so101_v1.stl"/>
+        <mesh filename="model://arm_description/assets/wrist_roll_follower_so101_v1.stl"/>
       </geometry>
     </collision>
@@ -307,5 +307,5 @@
       <origin xyz="-5.55112e-17 -5.55112e-17 0.0189" rpy="9.53145e-17 6.93889e-18 1.24077e-24"/>
       <geometry>
-        <mesh filename="package://arm_description/assets/moving_jaw_so101_v1.stl"/>
+        <mesh filename="model://arm_description/assets/moving_jaw_so101_v1.stl"/>
       </geometry>
       <material name="3d_printed"/>
@@ -314,5 +314,5 @@
       <origin xyz="-5.55112e-17 -5.55112e-17 0.0189" rpy="9.53145e-17 6.93889e-18 1.24077e-24"/>
       <geometry>
-        <mesh filename="package://arm_description/assets/moving_jaw_so101_v1.stl"/>
+        <mesh filename="model://arm_description/assets/moving_jaw_so101_v1.stl"/>
       </geometry>
     </collision>
