Commit message: added camera

File: src/arm_description/description/so101.urdf.xacro (robot description, xacro)
@@ -1,7 +1,8 @@
-<?xml version="1.0" encoding="utf-8"?>
-<!-- Generated using onshape-to-robot -->
-<!-- Onshape https://cad.onshape.com/documents/7715cc284bb430fe6dab4ffd/w/4fd0791b683777b02f8d975a/e/826c553ede3b7592eb9ca800 -->
-<robot name="so101_new_calib">
+<?xml version="1.0"?>
+<robot name="so101_new_calib" xmlns:xacro="http://www.ros.org/wiki/xacro">
+  <xacro:include filename="$(find arm_description)/description/camera.xacro"/>
+  <!-- ======================= -->
   <!-- Materials -->
+  <!-- ======================= -->
   <material name="3d_printed">
     <color rgba="1.0 0.82 0.12 1.0"/>
@@ -10,277 +11,178 @@
     <color rgba="0.1 0.1 0.1 1.0"/>
   </material>
-  <!-- Link base -->
+  <!-- ======================= -->
+  <!-- Macros -->
+  <!-- ======================= -->
+  <xacro:macro name="mesh_geom" params="file">
+    <geometry>
+      <mesh filename="model://arm_description/assets/${file}"/>
+    </geometry>
+  </xacro:macro>
+  <xacro:macro name="visual_mesh" params="xyz rpy file material">
+    <visual>
+      <origin xyz="${xyz}" rpy="${rpy}"/>
+      <xacro:mesh_geom file="${file}"/>
+      <material name="${material}"/>
+    </visual>
+  </xacro:macro>
+  <xacro:macro name="collision_mesh" params="xyz rpy file">
+    <collision>
+      <origin xyz="${xyz}" rpy="${rpy}"/>
+      <xacro:mesh_geom file="${file}"/>
+    </collision>
+  </xacro:macro>
+  <xacro:macro name="part" params="xyz rpy file material">
+    <xacro:visual_mesh xyz="${xyz}" rpy="${rpy}" file="${file}" material="${material}"/>
+    <xacro:collision_mesh xyz="${xyz}" rpy="${rpy}" file="${file}"/>
+  </xacro:macro>
+  <xacro:macro name="inertial_block" params="xyz mass ixx ixy ixz iyy iyz izz">
+    <inertial>
+      <origin xyz="${xyz}" rpy="0 0 0"/>
+      <mass value="${mass}"/>
+      <inertia
+        ixx="${ixx}" ixy="${ixy}" ixz="${ixz}"
+        iyy="${iyy}" iyz="${iyz}" izz="${izz}"/>
+    </inertial>
+  </xacro:macro>
+  <xacro:macro name="revolute_joint" params="name parent child xyz rpy axis lower upper effort velocity">
+    <joint name="${name}" type="revolute">
+      <origin xyz="${xyz}" rpy="${rpy}"/>
+      <parent link="${parent}"/>
+      <child link="${child}"/>
+      <axis xyz="${axis}"/>
+      <limit effort="${effort}" velocity="${velocity}" lower="${lower}" upper="${upper}"/>
+    </joint>
+  </xacro:macro>
+  <!-- ======================= -->
+  <!-- Links -->
+  <!-- ======================= -->
   <link name="base_link">
-    <inertial>
-      <origin xyz="0.0137179 -5.19711e-05 0.0334843" rpy="0 0 0"/>
-      <mass value="0.147"/>
-      <inertia ixx="0.000114686" ixy="-4.59787e-07" ixz="4.97151e-06" iyy="0.000136117" iyz="9.75275e-08" izz="0.000130364"/>
-    </inertial>
-    <!-- Part base_motor_holder_so101_v1 -->
-    <visual>
-      <origin xyz="-0.00636471 -9.94414e-05 -0.0024" rpy="1.5708 -1.67685e-15 1.5708"/>
-      <geometry>
-        <mesh filename="model://arm_description/assets/base_motor_holder_so101_v1.stl"/>
-      </geometry>
-      <material name="3d_printed"/>
-    </visual>
-    <collision>
-      <origin xyz="-0.00636471 -9.94414e-05 -0.0024" rpy="1.5708 -1.67685e-15 1.5708"/>
-      <geometry>
-        <mesh filename="model://arm_description/assets/base_motor_holder_so101_v1.stl"/>
-      </geometry>
-    </collision>
-    <!-- Part base_so101_v2 -->
-    <visual>
-      <origin xyz="-0.00636471 -8.97657e-09 -0.0024" rpy="1.5708 -2.78073e-29 1.5708"/>
-      <geometry>
-        <mesh filename="model://arm_description/assets/base_so101_v2.stl"/>
-      </geometry>
-      <material name="3d_printed"/>
-    </visual>
-    <collision>
-      <origin xyz="-0.00636471 -8.97657e-09 -0.0024" rpy="1.5708 -2.78073e-29 1.5708"/>
-      <geometry>
-        <mesh filename="model://arm_description/assets/base_so101_v2.stl"/>
-      </geometry>
-    </collision>
-    <!-- Part sts3215_03a_v1 -->
-    <visual>
-      <origin xyz="0.0263353 -8.97657e-09 0.0437" rpy="-8.21148e-16 7.84513e-18 1.249e-15"/>
-      <geometry>
-        <mesh filename="model://arm_description/assets/sts3215_03a_v1.stl"/>
-      </geometry>
-      <material name="sts3215"/>
-    </visual>
-    <collision>
-      <origin xyz="0.0263353 -8.97657e-09 0.0437" rpy="-8.21148e-16 7.84513e-18 1.249e-15"/>
-      <geometry>
-        <mesh filename="model://arm_description/assets/sts3215_03a_v1.stl"/>
-      </geometry>
-    </collision>
-    <!-- Part waveshare_mounting_plate_so101_v2 -->
-    <visual>
-      <origin xyz="-0.0309827 -0.000199441 0.0474" rpy="1.5708 -1.35493e-14 1.5708"/>
-      <geometry>
-        <mesh filename="model://arm_description/assets/waveshare_mounting_plate_so101_v2.stl"/>
-      </geometry>
-      <material name="3d_printed"/>
-    </visual>
-    <collision>
-      <origin xyz="-0.0309827 -0.000199441 0.0474" rpy="1.5708 -1.35493e-14 1.5708"/>
-      <geometry>
-        <mesh filename="model://arm_description/assets/waveshare_mounting_plate_so101_v2.stl"/>
-      </geometry>
-    </collision>
-  </link>
-  <!-- Link shoulder -->
+    <xacro:inertial_block
+      xyz="0.0137179 -5.19711e-05 0.0334843"
+      mass="0.147"
+      ixx="0.000114686" ixy="-4.59787e-07" ixz="4.97151e-06"
+      iyy="0.000136117" iyz="9.75275e-08" izz="0.000130364"/>
+    <xacro:part
+      xyz="-0.00636471 -9.94414e-05 -0.0024"
+      rpy="1.5708 -1.67685e-15 1.5708"
+      file="base_motor_holder_so101_v1.stl"
+      material="3d_printed"/>
+    <xacro:part
+      xyz="-0.00636471 -8.97657e-09 -0.0024"
+      rpy="1.5708 -2.78073e-29 1.5708"
+      file="base_so101_v2.stl"
+      material="3d_printed"/>
+    <xacro:part
+      xyz="0.0263353 -8.97657e-09 0.0437"
+      rpy="-8.21148e-16 7.84513e-18 1.249e-15"
+      file="sts3215_03a_v1.stl"
+      material="sts3215"/>
+    <xacro:part
+      xyz="-0.0309827 -0.000199441 0.0474"
+      rpy="1.5708 -1.35493e-14 1.5708"
+      file="waveshare_mounting_plate_so101_v2.stl"
+      material="3d_printed"/>
+  </link>
+  <link name="world"/>
+  <joint name="world_to_base" type="fixed">
+    <parent link="world"/>
+    <child link="base_link"/>
+    <origin xyz="0 0 -0.2" rpy="0 0 0"/>
+  </joint>
   <link name="shoulder_link">
-    <inertial>
-      <origin xyz="-0.0307604 -1.66727e-05 -0.0252713" rpy="0 0 0"/>
-      <mass value="0.100006"/>
-      <inertia ixx="8.3759e-05" ixy="7.55525e-08" ixz="-1.16342e-06" iyy="8.10403e-05" iyz="1.54663e-07" izz="2.39783e-05"/>
-    </inertial>
-    <!-- Part sts3215_03a_v1_2 -->
-    <visual>
-      <origin xyz="-0.0303992 0.000422241 -0.0417" rpy="1.5708 1.5708 0"/>
-      <geometry>
-        <mesh filename="model://arm_description/assets/sts3215_03a_v1.stl"/>
-      </geometry>
-      <material name="sts3215"/>
-    </visual>
-    <collision>
-      <origin xyz="-0.0303992 0.000422241 -0.0417" rpy="1.5708 1.5708 0"/>
-      <geometry>
-        <mesh filename="model://arm_description/assets/sts3215_03a_v1.stl"/>
-      </geometry>
-    </collision>
-    <!-- Part motor_holder_so101_base_v1 -->
-    <visual>
-      <origin xyz="-0.0675992 -0.000177759 0.0158499" rpy="1.5708 -1.5708 0"/>
-      <geometry>
-        <mesh filename="model://arm_description/assets/motor_holder_so101_base_v1.stl"/>
-      </geometry>
-      <material name="3d_printed"/>
-    </visual>
-    <collision>
-      <origin xyz="-0.0675992 -0.000177759 0.0158499" rpy="1.5708 -1.5708 0"/>
-      <geometry>
-        <mesh filename="model://arm_description/assets/motor_holder_so101_base_v1.stl"/>
-      </geometry>
-    </collision>
-    <!-- Part rotation_pitch_so101_v1 -->
-    <visual>
-      <origin xyz="0.0122008 2.22413e-05 0.0464" rpy="-1.5708 2.35221e-33 0"/>
-      <geometry>
-        <mesh filename="model://arm_description/assets/rotation_pitch_so101_v1.stl"/>
-      </geometry>
-      <material name="3d_printed"/>
-    </visual>
-    <collision>
-      <origin xyz="0.0122008 2.22413e-05 0.0464" rpy="-1.5708 2.35221e-33 0"/>
-      <geometry>
-        <mesh filename="model://arm_description/assets/rotation_pitch_so101_v1.stl"/>
-      </geometry>
-    </collision>
-  </link>
-  <!-- Link upper_arm -->
+    <xacro:inertial_block
+      xyz="-0.0307604 -1.66727e-05 -0.0252713"
+      mass="0.100006"
+      ixx="8.3759e-05" ixy="7.55525e-08" ixz="-1.16342e-06"
+      iyy="8.10403e-05" iyz="1.54663e-07" izz="2.39783e-05"/>
+    <xacro:part
+      xyz="-0.0303992 0.000422241 -0.0417"
+      rpy="1.5708 1.5708 0"
+      file="sts3215_03a_v1.stl"
+      material="sts3215"/>
+    <xacro:part
+      xyz="-0.0675992 -0.000177759 0.0158499"
+      rpy="1.5708 -1.5708 0"
+      file="motor_holder_so101_base_v1.stl"
+      material="3d_printed"/>
+    <xacro:part
+      xyz="0.0122008 2.22413e-05 0.0464"
+      rpy="-1.5708 2.35221e-33 0"
+      file="rotation_pitch_so101_v1.stl"
+      material="3d_printed"/>
+  </link>
   <link name="upper_arm_link">
-    <inertial>
-      <origin xyz="-0.0898471 -0.00838224 0.0184089" rpy="0 0 0"/>
-      <mass value="0.103"/>
-      <inertia ixx="4.08002e-05" ixy="-1.97819e-05" ixz="-4.03016e-08" iyy="0.000147318" iyz="8.97326e-09" izz="0.000142487"/>
-    </inertial>
-    <!-- Part sts3215_03a_v1_3 -->
-    <visual>
-      <origin xyz="-0.11257 -0.0155 0.0187" rpy="-3.14159 -5.27356e-16 -1.5708"/>
-      <geometry>
-        <mesh filename="model://arm_description/assets/sts3215_03a_v1.stl"/>
-      </geometry>
-      <material name="sts3215"/>
-    </visual>
-    <collision>
-      <origin xyz="-0.11257 -0.0155 0.0187" rpy="-3.14159 -5.27356e-16 -1.5708"/>
-      <geometry>
-        <mesh filename="model://arm_description/assets/sts3215_03a_v1.stl"/>
-      </geometry>
-    </collision>
-    <!-- Part upper_arm_so101_v1 -->
-    <visual>
-      <origin xyz="-0.065085 0.012 0.0182" rpy="3.14159 -0 -1.30911e-30"/>
-      <geometry>
-        <mesh filename="model://arm_description/assets/upper_arm_so101_v1.stl"/>
-      </geometry>
-      <material name="3d_printed"/>
-    </visual>
-    <collision>
-      <origin xyz="-0.065085 0.012 0.0182" rpy="3.14159 -0 -1.30911e-30"/>
-      <geometry>
-        <mesh filename="model://arm_description/assets/upper_arm_so101_v1.stl"/>
-      </geometry>
-    </collision>
-  </link>
-  <!-- Link lower_arm -->
+    <xacro:inertial_block
+      xyz="-0.0898471 -0.00838224 0.0184089"
+      mass="0.103"
+      ixx="4.08002e-05" ixy="-1.97819e-05" ixz="-4.03016e-08"
+      iyy="0.000147318" iyz="8.97326e-09" izz="0.000142487"/>
+    <xacro:part
+      xyz="-0.11257 -0.0155 0.0187"
+      rpy="-3.14159 -5.27356e-16 -1.5708"
+      file="sts3215_03a_v1.stl"
+      material="sts3215"/>
+    <xacro:part
+      xyz="-0.065085 0.012 0.0182"
+      rpy="3.14159 -0 -1.30911e-30"
+      file="upper_arm_so101_v1.stl"
+      material="3d_printed"/>
+  </link>
   <link name="lower_arm_link">
-    <inertial>
-      <origin xyz="-0.0980701 0.00324376 0.0182831" rpy="0 0 0"/>
-      <mass value="0.104"/>
-      <inertia ixx="2.87438e-05" ixy="7.41152e-06" ixz="1.26409e-06" iyy="0.000159844" iyz="-4.90188e-08" izz="0.00014529"/>
-    </inertial>
-    <!-- Part under_arm_so101_v1 -->
-    <visual>
-      <origin xyz="-0.0648499 -0.032 0.0182" rpy="3.14159 -0 6.67202e-31"/>
-      <geometry>
-        <mesh filename="model://arm_description/assets/under_arm_so101_v1.stl"/>
-      </geometry>
-      <material name="3d_printed"/>
-    </visual>
-    <collision>
-      <origin xyz="-0.0648499 -0.032 0.0182" rpy="3.14159 -0 6.67202e-31"/>
-      <geometry>
-        <mesh filename="model://arm_description/assets/under_arm_so101_v1.stl"/>
-      </geometry>
-    </collision>
-    <!-- Part motor_holder_so101_wrist_v1 -->
-    <visual>
-      <origin xyz="-0.0648499 -0.032 0.018" rpy="-3.14159 -2.55351e-15 -1.83387e-30"/>
-      <geometry>
-        <mesh filename="model://arm_description/assets/motor_holder_so101_wrist_v1.stl"/>
-      </geometry>
-      <material name="3d_printed"/>
-    </visual>
-    <collision>
-      <origin xyz="-0.0648499 -0.032 0.018" rpy="-3.14159 -2.55351e-15 -1.83387e-30"/>
-      <geometry>
-        <mesh filename="model://arm_description/assets/motor_holder_so101_wrist_v1.stl"/>
-      </geometry>
-    </collision>
-    <!-- Part sts3215_03a_v1_4 -->
-    <visual>
-      <origin xyz="-0.1224 0.0052 0.0187" rpy="-3.14159 -7.88861e-31 -3.14159"/>
-      <geometry>
-        <mesh filename="model://arm_description/assets/sts3215_03a_v1.stl"/>
-      </geometry>
-      <material name="sts3215"/>
-    </visual>
-    <collision>
-      <origin xyz="-0.1224 0.0052 0.0187" rpy="-3.14159 -7.88861e-31 -3.14159"/>
-      <geometry>
-        <mesh filename="model://arm_description/assets/sts3215_03a_v1.stl"/>
-      </geometry>
-    </collision>
-  </link>
-  <!-- Link wrist -->
+    <xacro:inertial_block
+      xyz="-0.0980701 0.00324376 0.0182831"
+      mass="0.104"
+      ixx="2.87438e-05" ixy="7.41152e-06" ixz="1.26409e-06"
+      iyy="0.000159844" iyz="-4.90188e-08" izz="0.00014529"/>
+    <xacro:part
+      xyz="-0.0648499 -0.032 0.0182"
+      rpy="3.14159 -0 6.67202e-31"
+      file="under_arm_so101_v1.stl"
+      material="3d_printed"/>
+    <xacro:part
+      xyz="-0.0648499 -0.032 0.018"
+      rpy="-3.14159 -2.55351e-15 -1.83387e-30"
+      file="motor_holder_so101_wrist_v1.stl"
+      material="3d_printed"/>
+    <xacro:part
+      xyz="-0.1224 0.0052 0.0187"
+      rpy="-3.14159 -7.88861e-31 -3.14159"
+      file="sts3215_03a_v1.stl"
+      material="sts3215"/>
+  </link>
   <link name="wrist_link">
-    <inertial>
-      <origin xyz="-0.000103312 -0.0386143 0.0281156" rpy="0 0 0"/>
-      <mass value="0.079"/>
-      <inertia ixx="3.68263e-05" ixy="1.7893e-08" ixz="-5.28128e-08" iyy="2.5391e-05" iyz="3.6412e-06" izz="2.1e-05"/>
-    </inertial>
-    <!-- Part sts3215_03a_no_horn_v1 -->
-    <visual>
-      <origin xyz="8.32667e-17 -0.0424 0.0306" rpy="1.5708 1.5708 0"/>
-      <geometry>
-        <mesh filename="model://arm_description/assets/sts3215_03a_no_horn_v1.stl"/>
-      </geometry>
-      <material name="sts3215"/>
-    </visual>
-    <collision>
-      <origin xyz="8.32667e-17 -0.0424 0.0306" rpy="1.5708 1.5708 0"/>
-      <geometry>
-        <mesh filename="model://arm_description/assets/sts3215_03a_no_horn_v1.stl"/>
-      </geometry>
-    </collision>
-    <!-- Part wrist_roll_pitch_so101_v2 -->
-    <visual>
-      <origin xyz="0 -0.028 0.0181" rpy="-1.5708 -1.5708 0"/>
-      <geometry>
-        <mesh filename="model://arm_description/assets/wrist_roll_pitch_so101_v2.stl"/>
-      </geometry>
-      <material name="3d_printed"/>
-    </visual>
-    <collision>
-      <origin xyz="0 -0.028 0.0181" rpy="-1.5708 -1.5708 0"/>
-      <geometry>
-        <mesh filename="model://arm_description/assets/wrist_roll_pitch_so101_v2.stl"/>
-      </geometry>
-    </collision>
-  </link>
-  <!-- Link gripper -->
+    <xacro:inertial_block
+      xyz="-0.000103312 -0.0386143 0.0281156"
+      mass="0.079"
+      ixx="3.68263e-05" ixy="1.7893e-08" ixz="-5.28128e-08"
+      iyy="2.5391e-05" iyz="3.6412e-06" izz="2.1e-05"/>
+    <xacro:part
+      xyz="8.32667e-17 -0.0424 0.0306"
+      rpy="1.5708 1.5708 0"
+      file="sts3215_03a_no_horn_v1.stl"
+      material="sts3215"/>
+    <xacro:part
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
Commit message: WIP: MoveIt + SmolVLA progress

File: src/arm_description/description/so101.urdf.xacro (robot description, xacro)
@@ -191,4 +191,23 @@
     </inertial>
   </link>
+  <!-- tcp_jaw_link: synthetic frame placed at the approximate jaw-close point
+       so MoveIt + local IK can plan pick poses that put the physical jaws, not
+       the (offset) gripper_frame_link, around the target object. Offsets were
+       derived from inspecting the fixed offsets of the stationary finger
+       (wrist_roll_follower_so101_v1 at gripper_link origin) and moving_jaw
+       origin (at +0.020, +0.019, -0.023 in gripper_link frame). Placed at the
+       midpoint and pushed outward along -Z (gripper's approach direction). -->
+  <link name="tcp_jaw_link">
+    <inertial>
+      <origin xyz="0 0 0" rpy="0 0 0"/>
+      <mass value="1e-9"/>
+      <inertia ixx="0" ixy="0" ixz="0" iyy="0" iyz="0" izz="0"/>
+    </inertial>
+  </link>
+  <joint name="tcp_jaw_joint" type="fixed">
+    <origin xyz="0.012 0.010 -0.035" rpy="0 0 0"/>
+    <parent link="gripper_link"/>
+    <child link="tcp_jaw_link"/>
+  </joint>
   <link name="moving_jaw_so101_v1_link">
     <xacro:inertial_block
@@ -325,4 +344,29 @@
       </ros>
     </plugin>
+    <!-- DetachableJoint plugins: one per graspable object. When an /attach_{color}
+         message is published (gz.msgs.Empty), a fixed joint is created between
+         gripper_link and that ball's link. /detach_{color} removes it. Used by the
+         expert policy to enforce reliable grasp during sim demo collection — the
+         VLA learns motion patterns, and physical-grasp realism isn't critical. -->
+    <plugin filename="gz-sim-detachable-joint-system"
+            name="gz::sim::systems::DetachableJoint">
+      <parent_link>gripper_link</parent_link>
+      <child_model>blue_ball</child_model>
+      <child_link>link</child_link>
+      <attach_topic>/attach_blue</attach_topic>
+      <detach_topic>/detach_blue</detach_topic>
+      <output_topic>/attach_blue_state</output_topic>
+      <suppress_child_warning>true</suppress_child_warning>
+    </plugin>
+    <plugin filename="gz-sim-detachable-joint-system"
+            name="gz::sim::systems::DetachableJoint">
+      <parent_link>gripper_link</parent_link>
+      <child_model>red_ball</child_model>
+      <child_link>link</child_link>
+      <attach_topic>/attach_red</attach_topic>
+      <detach_topic>/detach_red</detach_topic>
+      <output_topic>/attach_red_state</output_topic>
+      <suppress_child_warning>true</suppress_child_warning>
+    </plugin>
   </gazebo>
 </robot>
